Commit message: working

File: urdf/wamv_base.xacro (robot description, xacro)
@@ -5,19 +5,19 @@
     <visual>
      <geometry>
-       <mesh filename="package://wamv_description/mesh/blender/WAM-V-Base.dae"/>
+       <mesh filename="package://wamv_description/mesh/WAM-V-Base.dae"/>
      </geometry>
    </visual>
    <collision name="base_link_collision">
      <geometry>
-       <mesh filename="package://wamv_description/mesh/blender/WAM-V-Base.dae"/>
+       <mesh filename="package://wamv_description/mesh/WAM-V-Base.dae"/>
      </geometry>
    </collision>
    <inertial>
-     <mass value="247.07"/>
-     <inertia ixx="200" ixy="0.03" ixz="3.09" iyy="500" iyz="-0.05" izz="165.39"/>
+     <mass value="180.0"/> <!-- From von Ellenrieder -->
+     <inertia ixx="200.0" ixy="0.03" ixz="3.09" iyy="500" iyz="-0.05" izz="250.0"/>
    </inertial>
   </link>
   <joint name="base_link_joint" type="fixed">
-    <origin xyz="0 0 1.84"/>
+    <origin xyz="0 0 0"/>
     <parent link="base_footprint"/>
     <child link="base_link"/>

Commit message: towards waves

File: urdf/wamv_base.xacro (robot description, xacro)
@@ -3,4 +3,5 @@
   <xacro:include filename="properties.urdf.xacro"/>
   <link name="base_link">
+    <wind>true</wind>
     <visual>
      <geometry>
@@ -14,6 +15,7 @@
    </collision>
    <inertial>
-     <mass value="180.0"/> <!-- From von Ellenrieder -->
-     <inertia ixx="200.0" ixy="0.03" ixz="3.09" iyy="500" iyz="-0.05" izz="250.0"/>
+     <mass value="180.0"/> <!-- From von Ellenrieder, consistent with WAM-V specs-->
+     <!--<inertia ixx="200.0" ixy="0.03" ixz="3.09" iyy="500" iyz="-0.05" izz="250.0"/>-->
+     <inertia ixx="120.0" ixy="0.03" ixz="3.09" iyy="393" iyz="-0.05" izz="446.0"/>
    </inertial>
   </link>

Commit message: working, sloppy version

File: urdf/wamv_base.xacro (robot description, xacro)
@@ -17,5 +17,5 @@
      <mass value="180.0"/> <!-- From von Ellenrieder, consistent with WAM-V specs-->
      <!--<inertia ixx="200.0" ixy="0.03" ixz="3.09" iyy="500" iyz="-0.05" izz="250.0"/>-->
-     <inertia ixx="120.0" ixy="0.03" ixz="3.09" iyy="393" iyz="-0.05" izz="446.0"/>
+     <inertia ixx="120.0" ixy="0.0" ixz="0.0" iyy="393" iyz="0.0" izz="446.0"/>
    </inertial>
   </link>
